Commit message: feat: omni_robot 添加后相机，2d-ego-planner 适配 PID 跟踪器

File: src/omni_robot/omni_gazebo/urdf/omni_robot.xacro (robot description, xacro)
@@ -1,22 +1,23 @@
 <?xml version='1.0'?>
 <robot name="omni_robot" xmlns:xacro="http://www.ros.org/wiki/xacro">
-  	<xacro:include filename="$(find omni_gazebo)/urdf/omni_robot.gazebo" />
-	<xacro:property name="scale" value="0.01" />
-    <xacro:arg name="gpu" default="false"/>
-    <xacro:property name="gpu" value="$(arg gpu)" />
-    <xacro:arg name="organize_cloud" default="true"/>
-    <xacro:property name="organize_cloud" value="$(arg organize_cloud)" />
+	<xacro:include filename="$(find omni_gazebo)/urdf/omni_robot.gazebo" />
+	<xacro:property name="scale" value="10" />
+	<xacro:arg name="gpu" default="false" />
+	<xacro:property name="gpu" value="$(arg gpu)" />
+	<xacro:arg name="organize_cloud" default="true" />
+	<xacro:property name="organize_cloud" value="$(arg organize_cloud)" />
 	<xacro:property name="base_z_size" value="0.410000" />
-    <xacro:include filename="$(find omni_gazebo)/urdf/sensors/inertial.xacro" />
-    <xacro:include filename="$(find omni_gazebo)/urdf/sensors/laser_support.xacro" />
-    <xacro:include filename="$(find velodyne_description)/urdf/VLP-16.urdf.xacro"/>
-    <xacro:VLP-16 parent="support" name="velodyne" topic="/velodyne_points" organize_cloud="${organize_cloud}" hz="10" samples="400" gpu="${gpu}">
-          <origin xyz="0 0 ${support_length/4}" rpy="0 0 0" />
-    </xacro:VLP-16>
-    <xacro:include filename="$(find omni_gazebo)/urdf/sensors/imu.xacro"/>
-    <xacro:imu sensor_name="imu" parent_link="base_link">
-    <origin rpy="0 0 0" xyz="-0.03 0 ${base_z_size/2}"/>
-    </xacro:imu>
-  	<link name="base_footprint"></link>
+	<xacro:include filename="$(find omni_gazebo)/urdf/sensors/inertial.xacro" />
+	<xacro:include filename="$(find omni_gazebo)/urdf/sensors/laser_support.xacro" />
+	<xacro:include filename="$(find velodyne_description)/urdf/VLP-16.urdf.xacro" />
+	<xacro:VLP-16 parent="support" name="velodyne" topic="/velodyne_points"
+		organize_cloud="${organize_cloud}" hz="10" samples="400" gpu="${gpu}">
+		<origin xyz="0 0 ${support_length/4}" rpy="0 0 0" />
+	</xacro:VLP-16>
+	<xacro:include filename="$(find omni_gazebo)/urdf/sensors/imu.xacro" />
+	<xacro:imu sensor_name="imu" parent_link="base_link">
+		<origin rpy="0 0 0" xyz="-0.03 0 ${base_z_size/2}" />
+	</xacro:imu>
+	<link name="base_footprint"></link>
 	<joint name="robot_footprint_joint" type="fixed">
 		<origin xyz="0 0 0.07" rpy="0 0 0" />
@@ -29,9 +30,9 @@
 			<origin xyz="0 0 0" rpy="0 0 0" />
 			<geometry>
-				<cylinder radius="0.27" length="0.05"/>
+				<cylinder radius="0.27" length="0.05" />
 				<!--long,wide,tall-->
 			</geometry>
 			<material name="blue">
-				<color rgba="0 0.5 1 1"/>
+				<color rgba="0 0.5 1 1" />
 			</material>
 		</visual>
@@ -40,12 +41,12 @@
 			<origin xyz="0 0 0" rpy="0 0 0" />
 			<geometry>
-				<cylinder radius="0.27" length="0.05"/>
+				<cylinder radius="0.27" length="0.05" />
 				<!--long,wide,tall-->
 			</geometry>
 		</collision>
 		<inertial>
-			<mass value="${10.0*scale}"/>
+			<mass value="${10.0*scale}" />
 			<inertia ixx="0.5" ixy="0.0" ixz="0.0"
-					iyy="0.1391" iyz="0.0" izz="1.6125"/>
+				iyy="0.1391" iyz="0.0" izz="1.6125" />
 		</inertial>
 		<visual name="left_bottom_cylinder">
@@ -55,5 +56,5 @@
 			</geometry>
 			<material name="white">
-				<color rgba="0 0 0 1"/>
+				<color rgba="0 0 0 1" />
 			</material>
 		</visual>
@@ -65,5 +66,5 @@
 				<box size="0.02 0.02 0.25" />
 			</geometry>
-			<material name="white"/>
+			<material name="white" />
 		</visual>
 		<!-- between_top_cylinder -->
@@ -73,5 +74,5 @@
 				<box size="0.02 0.02 0.25" />
 			</geometry>
-			<material name="white"/>
+			<material name="white" />
 		</visual>
 		<!-- hold_box1 -->
@@ -81,5 +82,5 @@
 				<cylinder radius="0.25" length="0.05" />
 			</geometry>
-			<material name="blue"/>
+			<material name="blue" />
 		</visual>
 		<!-- hold_box2
@@ -95,17 +96,17 @@
 	<joint name="astra_joint" type="fixed">
 		<axis xyz="0 0 0" />
-		<origin xyz="0.15 0 0.33" rpy="0 0 0"/>
-		<parent link="base_link"/>
-		<child link="camera_link"/>
+		<origin xyz="0.20 0 0.33" rpy="0 0 0" />
+		<parent link="base_link" />
+		<child link="camera_link" />
 	</joint>
 	<link name="camera_link">
 		<collision>
-			<origin xyz="0 0 0" rpy="0 0 0"/>
-			<geometry>
-				<box size="0.001 0.001 0.001"/>
-			</geometry>
-		</collision>
-		<visual>
-			<origin xyz="-0.01 0 -0.03" rpy="1.5707 0 1.5707"/>
+			<origin xyz="0 0 0" rpy="0 0 0" />
+			<geometry>
+				<box size="0.001 0.001 0.001" />
+			</geometry>
+		</collision>
+		<visual>
+			<origin xyz="-0.01 0 -0.03" rpy="1.5707 0 1.5707" />
 			<geometry>
 				<mesh filename="package://omni_gazebo/meshes/astra.dae" scale="0.001 0.001 0.001" />
@@ -114,23 +115,64 @@
 		<inertial>
 			<mass value="${1e-5*scale}" />
-			<origin xyz="0 0 0" rpy="0 0 0"/>
+			<origin xyz="0 0 0" rpy="0 0 0" />
 			<inertia ixx="0" ixy="0" ixz="0" iyy="0" iyz="0" izz="0" />
 		</inertial>
 	</link>
 	<joint name="camera_optical_joint" type="fixed">
-		<origin xyz="0 0 0" rpy="0 0 0"/>
-		<parent link="camera_link"/>
-		<child link="camera_rgb_frame"/>
+		<origin xyz="0 0 0" rpy="0 0 0" />
+		<parent link="camera_link" />
+		<child link="camera_rgb_frame" />
 	</joint>
 	<link name="camera_rgb_frame">
 	</link>
 	<joint name="camera_depth_joint" type="fixed">
-		<origin xyz="0 0 0" rpy="-1.5707 0 -1.5707"/>
-		<parent link="camera_link"/>
-		<child link="camera_depth_frame"/>
+		<origin xyz="0 0 0" rpy="-1.5707 0 -1.5707" />
+		<parent link="camera_link" />
+		<child link="camera_depth_frame" />
 	</joint>
 	<link name="camera_depth_frame">
 	</link>
-	<!--<joint name="rplidar_joint" type="fixed">
+	<!-- back Orbbec Astra RGBD Camera -->
+	<joint name="astra_joint_back" type="fixed">
+		<axis xyz="0 0 0" />
+		<origin xyz="-0.20 0 0.33" rpy="0 0 3.14" />
+		<parent link="base_link" />
+		<child link="camera_link_back" />
+	</joint>
+	<link name="camera_link_back">
+		<collision>
+			<origin xyz="0 0 0" rpy="0 0 0" />
+			<geometry>
+				<box size="0.001 0.001 0.001" />
+			</geometry>
+		</collision>
+		<visual>
+			<origin xyz="-0.01 0 -0.03" rpy="1.5707 0 1.5707" />
+			<geometry>
+				<mesh filename="package://omni_gazebo/meshes/astra.dae" scale="0.001 0.001 0.001" />
+			</geometry>
+		</visual>
+		<inertial>
+			<mass value="${1e-5*scale}" />
+			<origin xyz="0 0 0" rpy="0 0 0" />
+			<inertia ixx="0" ixy="0" ixz="0" iyy="0" iyz="0" izz="0" />
+		</inertial>
+	</link>
+	<joint name="camera_optical_joint_back" type="fixed">
+		<origin xyz="0 0 0" rpy="0 0 0" />
+		<parent link="camera_link_back" />
+		<child link="camera_rgb_frame_back" />
+	</joint>
+	<link name="camera_rgb_frame_back">
+</link>
+	<joint name="camera_depth_joint_back" type="fixed">
+		<origin xyz="0 0 0" rpy="-1.5707 0 -1.5707" />
+		<parent link="camera_link_back" />
+		<child link="camera_depth_frame_back" />
+	</joint>
+	<link name="camera_depth_frame_back">
+</link>
+	<!--<joint
+	name="rplidar_joint" type="fixed">
 		<axis xyz="0 1 0" />
 		<origin xyz="0.02 0 0.530" rpy="0 0 0"/>
@@ -139,5 +181,6 @@
 	</joint>-->
 	<!-- rplidar Laser -->
-	<!--<link name="laser">
+	<!--<link
+	name="laser">
 		<collision>
 			<origin xyz="0 0 0" rpy="1.5707 0 3.1412"/>
@@ -159,5 +202,5 @@
 	</link>-->
 	<!-- IMU -->
-<!--
+	<!--
 	<joint name="imu_sensor_joint" type="continuous">
         <axis xyz="0 0 1" />
@@ -188,10 +231,10 @@
 	<!-- top_wheel -->
 	<joint name="joint_top_wheel" type="fixed">
-		<parent link="base_link"/>
-		<child link="top_wheel"/>
+		<parent link="base_link" />
+		<child link="top_wheel" />
 		<origin xyz="0.33 0 0" rpy="1.570796 0 1.570796" />
 		<axis xyz="0 0 1" />
 		<!-- <limit effort="100" velocity="100"/> -->
-		<joint_properties damping="0.0" friction="0.0"/>
+		<joint_properties damping="0.0" friction="0.0" />
 	</joint>
 	<transmission name="top_wheel_trans" type="SimpleTransmission">
@@ -208,8 +251,8 @@
 			<origin xyz="0 0 0" rpy="0 0 0.0" />
 			<geometry>
-				<mesh filename="package://omni_gazebo/meshes/rim.stl" scale="5 5 5"/>
+				<mesh filename="package://omni_gazebo/meshes/rim.stl" scale="5 5 5" />
 			</geometry>
 			<material name="left_rim_material">
-				<color rgba="0.3 0 0 1"/>
+				<color rgba="0.3 0 0 1" />
 			</material>
 		</visual>
@@ -217,21 +260,21 @@
 		<collision>
 			<geometry>
-				<mesh filename="package://omni_gazebo/meshes/rim.stl" scale="5 5 5"/>
-			</geometry>
-		</collision>
-		<inertial>
-			<mass value="${5*scale}"/>
+				<mesh filename="package://omni_gazebo/meshes/rim.stl" scale="5 5 5" />
+			</geometry>
+		</collision>
+		<inertial>
+			<mass value="${5*scale}" />
 			<inertia ixx="0.070416667" ixy="0" ixz="0"
-					iyy="0.0325" iyz="0" izz="0.070416667"/>
+				iyy="0.0325" iyz="0" izz="0.070416667" />
 		</inertial>
 	</link>
 	<!-- right_bottom Wheel -->
 	<joint name="joint_right_bottom_wheel" type="fixed">
-		<parent link="base_link"/>
-		<child link="right_bottom_wheel"/>
+		<parent link="base_link" />
+		<child link="right_bottom_wheel" />
 		<origin xyz="-0.165 0.285788 0" rpy="1.570795 0 -2.61799" />
 		<axis xyz="0 0 1" />
 		<!-- <limit effort="100" velocity="100"/> -->
-		<joint_properties damping="0.0" friction="0.0"/>
+		<joint_properties damping="0.0" friction="0.0" />
 	</joint>
 	<transmission name="right_bottom_wheel_trans" type="SimpleTransmission">
@@ -246,32 +289,32 @@
 	<link name="right_bottom_wheel">
 		<visual>
-		<origin xyz="0 0 0" rpy="0 0 0.0" />
-		<geometry>
-			<mesh filename="package://omni_gazebo/meshes/rim.stl" scale="5 5 5"/>
-		</geometry>
-		<material name="left_rim_material">
-			<color rgba="0.3 0 0 1"/>
-		</material>
+			<origin xyz="0 0 0" rpy="0 0 0.0" />
+			<geometry>
+				<mesh filename="package://omni_gazebo/meshes/rim.stl" scale="5 5 5" />
+			</geometry>
+			<material name="left_rim_material">
+				<color rgba="0.3 0 0 1" />
+			</material>
 		</visual>
 		<!-- right_bottom_wheel collision -->
 		<collision>
 			<geometry>
-				<mesh filename="package://omni_gazebo/meshes/rim.stl" scale="5 5 5"/>
-			</geometry>
-		</collision>
-		<inertial>
-			<mass value="${5*scale}"/>
+				<mesh filename="package://omni_gazebo/meshes/rim.stl" scale="5 5 5" />
+			</geometry>
+		</collision>
+		<inertial>
+			<mass value="${5*scale}" />
 			<inertia ixx="0.070416667" ixy="0" ixz="0"
-					iyy="0.0325" iyz="0" izz="0.070416667"/>
+				iyy="0.0325" iyz="0" izz="0.070416667" />
 		</inertial>
 	</link>
 	<!-- right left_bottom Wheel -->
 	<joint name="joint_left_bottom_wheel" type="fixed">
-		<parent link="base_link"/>
-		<child link="left_bottom_wheel"/>
+		<parent link="base_link" />
+		<child link="left_bottom_wheel" />
 		<origin xyz="-0.165 -0.285788 0" rpy="1.570795 0 -0.52360" />
 		<axis xyz="0 0 1" />
 		<!-- <limit effort="100" velocity="100"/> -->
-		<joint_properties damping="0.0" friction="0.0"/>
+		<joint_properties damping="0.0" friction="0.0" />
 	</joint>
 	<transmission name="left_bottom_wheel_trans" type="SimpleTransmission">
@@ -285,11 +328,11 @@
 	</transmission>
 	<link name="left_bottom_wheel">
-	<visual>
-		<origin xyz="0 0 0" rpy="0 0 0.0" />
-		<geometry>
-			<mesh filename="package://omni_gazebo/meshes/rim.stl" scale="5 5 5"/>
-		</geometry>
+		<visual>
+			<origin xyz="0 0 0" rpy="0 0 0.0" />
+			<geometry>
+				<mesh filename="package://omni_gazebo/meshes/rim.stl" scale="5 5 5" />
+			</geometry>
 			<material name="left_rim_material">
-				<color rgba="0.3 0 0 1"/>
+				<color rgba="0.3 0 0 1" />
 			</material>
 		</visual>
@@ -297,11 +340,11 @@
 		<collision>
 			<geometry>
-				<mesh filename="package://omni_gazebo/meshes/rim.stl" scale="5 5 5"/>
-			</geometry>
-		</collision>
-		<inertial>
-			<mass value="${5*scale}"/>
+				<mesh filename="package://omni_gazebo/meshes/rim.stl" scale="5 5 5" />
+			</geometry>
+		</collision>
+		<inertial>
+			<mass value="${5*scale}" />
 			<inertia ixx="0.070416667" ixy="0" ixz="0"
-					iyy="0.0325" iyz="0" izz="0.070416667"/>
+				iyy="0.0325" iyz="0" izz="0.070416667" />
 		</inertial>
 	</link>
@@ -310,26 +353,26 @@
 	<link name="bottem_left_roller_e_link">
 		<visual>
-			<origin xyz="0 0 0" rpy="0 0 0"/>
-			<geometry>
-				<mesh filename="package://omni_gazebo/meshes/roller.stl" scale="5 5 5"/>
+			<origin xyz="0 0 0" rpy="0 0 0" />
+			<geometry>
+				<mesh filename="package://omni_gazebo/meshes/roller.stl" scale="5 5 5" />
 			</geometry>
 			<material name="bottem_left_roller_e_material">
-				<color rgba="0.0 0.0 1.0 1"/>
-			</material>
-		</visual>
-		<inertial>
-			<mass value="${0.00179*scale}"/>
-			<inertia
-				ixx="0.000005"
-				ixy="0"
-				ixz="0"
-				iyy="0.000005"
-				iyz="0"
-				izz="0.000003"
-			/>
-		</inertial>
-		<collision>
-			<geometry>
-				<mesh filename="package://omni_gazebo/meshes/roller.stl" scale="5 5 5"/>
+				<color rgba="0.0 0.0 1.0 1" />
+			</material>
+		</visual>
+		<inertial>
+			<mass value="${0.00179*scale}" />
+			<inertia
+				ixx="0.000005"
+				ixy="0"
+				ixz="0"
+				iyy="0.000005"
+				iyz="0"
+				izz="0.000003"
+			/>
+		</inertial>
+		<collision>
+			<geometry>
+				<mesh filename="package://omni_gazebo/meshes/roller.stl" scale="5 5 5" />
 			</geometry>
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
Commit message: feat: 更改车体模型模仿人的体型

File: src/omni_robot/omni_gazebo/urdf/omni_robot.xacro (robot description, xacro)
@@ -80,8 +80,14 @@
 			<origin xyz="0 0 0.26" rpy="0 0 0" />
 			<geometry>
-				<cylinder radius="0.25" length="0.05" />
-			</geometry>
-			<material name="blue" />
-		</visual>
+				<box size="0.55 1.00 0.05" />
+			</geometry>
+			<material name="white" />
+		</visual>
+		<collision name="hold_box1">
+			<origin xyz="0 0 0" rpy="0 0 0" />
+			<geometry>
+				<box size="0.55 1.00 0.05" />
+			</geometry>
+		</collision>
 		<!-- hold_box2
 		<visual name="hold_box2">

Commit message: feat: 定义轨迹跟踪器类并集成进 ego-planner 主节点中

File: src/omni_robot/omni_gazebo/urdf/omni_robot.xacro (robot description, xacro)
@@ -76,18 +76,4 @@
 			<material name="white" />
 		</visual>
-		<!-- hold_box1 -->
-		<visual name="hold_box1">
-			<origin xyz="0 0 0.26" rpy="0 0 0" />
-			<geometry>
-				<box size="0.55 1.00 0.05" />
-			</geometry>
-			<material name="white" />
-		</visual>
-		<collision name="hold_box1">
-			<origin xyz="0 0 0" rpy="0 0 0" />
-			<geometry>
-				<box size="0.55 1.00 0.05" />
-			</geometry>
-		</collision>
 		<!-- hold_box2
 		<visual name="hold_box2">
@@ -99,4 +85,26 @@
 		</visual> -->
 	</link>
+	<link name="hold_box1">
+		<visual name="hold_box1">
+			<geometry>
+				<box size="0.55 1.00 0.05" />
+			</geometry>
+			<material name="blue">
+				<color rgba="0 0 1 1" />
+			</material>
+		</visual>
+		<collision name="hold_box1">
+			<origin xyz="0 0 0" rpy="0 0 0" />
+			<geometry>
+				<box size="0.55 1.00 0.05" />
+			</geometry>
+		</collision>
+	</link>
+	<joint name="hold_box1_joint" type="fixed">
+		<axis xyz="0 0 0" />
+		<origin xyz="0 0 0.26" rpy="0 0 0" />
+		<parent link="base_link" />
+		<child link="hold_box1" />
+	</joint>
 	<!-- Orbbec Astra RGBD Camera -->
 	<joint name="astra_joint" type="fixed">
